Commit message: Moved files to gypsy_ros and gypsy_gazebo

File: urdf/gypsy.xacro (robot description, xacro)
@@ -4,12 +4,12 @@
   <!--xacro:include filename="$(find mybot_description)/urdf/materials.xacro" /-->
   <!--xacro:include filename="$(find mybot_description)/urdf/macros.xacro" /-->
-  <link name="chassis">
+  <link name="base_link">
     <visual>
       <geometry>
-        <!--cylinder length="0.0508" radius="0.1524" /-->
-	<mesh filename="package://gypsy_description/meshes/gypsy_frame.dae"/>
+        <cylinder length="0.0508" radius="0.1524" />
+	<!--mesh filename="package://gypsy_description/meshes/gypsy_frame.dae"/-->
       </geometry>
       <material name="plastic">
-        <color rgba="0 1 0 0" />
+        <color rgba="1 1 1 1" />
       </material>
     </visual>
@@ -50,5 +50,5 @@
   </link>
   <joint name="right_wheel_joint" type="continuous">
-    <parent link="chassis" />
+    <parent link="base_link" />
     <child link="right_wheel" />
     <origin xyz="0 -0.168402 0" rpy="1.57075 0 0" />
@@ -78,5 +78,5 @@
   </link>
   <joint name="left_wheel_joint" type="continuous">
-    <parent link="chassis" />
+    <parent link="base_link" />
     <child link="left_wheel" />
     <origin xyz="0 0.168402 0" rpy="1.57075 0 0" />

Commit message: Corrected axis of wheels for correct turning direction.

File: urdf/gypsy.xacro (robot description, xacro)
@@ -1,5 +1,4 @@
 <?xml version="1.0"?>
 <robot name="gypsy" xmlns:xacro="http://www.ros.org/wiki/xacro">
-  <xacro:include filename="$(find gypsy_description)/urdf/gypsy.gazebo" />
   <!--xacro:include filename="$(find mybot_description)/urdf/materials.xacro" /-->
   <!--xacro:include filename="$(find mybot_description)/urdf/macros.xacro" /-->
@@ -52,5 +51,5 @@
     <parent link="base_link" />
     <child link="right_wheel" />
-    <origin xyz="0 -0.168402 0" rpy="1.57075 0 0" />
+    <origin xyz="0 -0.168402 0" rpy="-1.57075 0 0" />
     <axis xyz="0 0 1" />
     <limit effort="100" velocity="100"/>
@@ -80,5 +79,5 @@
     <parent link="base_link" />
     <child link="left_wheel" />
-    <origin xyz="0 0.168402 0" rpy="1.57075 0 0" />
+    <origin xyz="0 +0.168402 0" rpy="-1.57075 0 0" />
     <axis xyz="0 0 1" />
     <limit effort="100" velocity="100"/>
